File: Synthesizer/Synthesizer.kicad_pcb (KiCad board)
At the start: 2 copper layers, 18 parts, among them Q1 BC108, Q2 BC108, U1 LM358, U2 Teensy3.6

Commit message: Add buffer for fuzz
Parts:
- added U3: TL071, Package_DIP:DIP-8_W7.62mm_Socket, F.Cu at (34.3, 48.3)
Connections:
- FUZZ_IN1 pad 2: Net-(C1-Pad2) -> Net-(FUZZ_IN1-Pad2)
Changed lines of the file:
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@@
     (tracks 0)
     (zones 0)
-    (modules 18)
-    (nets 101)
+    (modules 19)
+    (nets 105)
   )
   (page A4)
@@
   (net 99 "Net-(U2-Pad1)")
   (net 100 "Net-(FUZZ_GAIN1-Pad1)")
+  (net 101 "Net-(U3-Pad1)")
+  (net 102 "Net-(U3-Pad5)")
+  (net 103 "Net-(FUZZ_IN1-Pad2)")
+  (net 104 "Net-(U3-Pad8)")
   (net_class Default "This is the default net class."
     (clearance 0.2)
@@
     (add_net "Net-(C3-Pad1)")
     (add_net "Net-(FUZZ_GAIN1-Pad1)")
+    (add_net "Net-(FUZZ_IN1-Pad2)")
     (add_net "Net-(Q1-Pad3)")
     (add_net "Net-(Q2-Pad3)")
@@
     (add_net "Net-(U2-Pad86)")
     (add_net "Net-(U2-Pad9)")
+    (add_net "Net-(U3-Pad1)")
+    (add_net "Net-(U3-Pad5)")
+    (add_net "Net-(U3-Pad8)")
+  )
+  (module Package_DIP:DIP-8_W7.62mm_Socket (layer F.Cu)
+    (at 34.29 48.26)
+    (descr "8-lead though-hole mounted DIP package, row spacing 7.62 mm (300 mils), Socket")
+    (tags "THT DIP DIL PDIP 2.54mm 7.62mm 300mil Socket")
+    (fp_text reference U3 (at 3.81 -2.33) (layer F.SilkS)
+      (effects (font (size 1 1) (thickness 0.15)))
+    )
+    (fp_text value TL071 (at 3.81 9.95) (layer F.Fab)
+      (effects (font (size 1 1) (thickness 0.15)))
+    )
+    (fp_arc (start 3.81 -1.33) (end 2.81 -1.33) (angle -180) (layer F.SilkS) (width 0.12))
+    (fp_line (start 1.635 -1.27) (end 6.985 -1.27) (layer F.Fab) (width 0.1))
+    (fp_line (start 6.985 -1.27) (end 6.985 8.89) (layer F.Fab) (width 0.1))
+    (fp_line (start 6.985 8.89) (end 0.635 8.89) (layer F.Fab) (width 0.1))
+    (fp_line (start 0.635 8.89) (end 0.635 -0.27) (layer F.Fab) (width 0.1))
+    (fp_line (start 0.635 -0.27) (end 1.635 -1.27) (layer F.Fab) (width 0.1))
+    (fp_line (start -1.27 -1.33) (end -1.27 8.95) (layer F.Fab) (width 0.1))
+    (fp_line (start -1.27 8.95) (end 8.89 8.95) (layer F.Fab) (width 0.1))
+    (fp_line (start 8.89 8.95) (end 8.89 -1.33) (layer F.Fab) (width 0.1))
+    (fp_line (start 8.89 -1.33) (end -1.27 -1.33) (layer F.Fab) (width 0.1))
+    (fp_line (start 2.81 -1.33) (end 1.16 -1.33) (layer F.SilkS) (width 0.12))
+    (fp_line (start 1.16 -1.33) (end 1.16 8.95) (layer F.SilkS) (width 0.12))
+    (fp_line (start 1.16 8.95) (end 6.46 8.95) (layer F.SilkS) (width 0.12))
+    (fp_line (start 6.46 8.95) (end 6.46 -1.33) (layer F.SilkS) (width 0.12))
+    (fp_line (start 6.46 -1.33) (end 4.81 -1.33) (layer F.SilkS) (width 0.12))
+    (fp_line (start -1.33 -1.39) (end -1.33 9.01) (layer F.SilkS) (width 0.12))
+    (fp_line (start -1.33 9.01) (end 8.95 9.01) (layer F.SilkS) (width 0.12))
+    (fp_line (start 8.95 9.01) (end 8.95 -1.39) (layer F.SilkS) (width 0.12))
+    (fp_line (start 8.95 -1.39) (end -1.33 -1.39) (layer F.SilkS) (width 0.12))
+    (fp_line (start -1.55 -1.6) (end -1.55 9.2) (layer F.CrtYd) (width 0.05))
+    (fp_line (start -1.55 9.2) (end 9.15 9.2) (layer F.CrtYd) (width 0.05))
+    (fp_line (start 9.15 9.2) (end 9.15 -1.6) (layer F.CrtYd) (width 0.05))
+    (fp_line (start 9.15 -1.6) (end -1.55 -1.6) (layer F.CrtYd) (width 0.05))
+    (fp_text user %R (at 3.81 3.81) (layer F.Fab)
+      (effects (font (size 1 1) (thickness 0.15)))
+    )
+    (pad 1 thru_hole rect (at 0 0) (size 1.6 1.6) (drill 0.8) (layers *.Cu *.Mask)
+      (net 101 "Net-(U3-Pad1)"))
+    (pad 5 thru_hole oval (at 7.62 7.62) (size 1.6 1.6) (drill 0.8) (layers *.Cu *.Mask)
+      (net 102 "Net-(U3-Pad5)"))
+    (pad 2 thru_hole oval (at 0 2.54) (size 1.6 1.6) (drill 0.8) (layers *.Cu *.Mask)
+      (net 2 "Net-(C1-Pad2)"))
+    (pad 6 thru_hole oval (at 7.62 5.08) (size 1.6 1.6) (drill 0.8) (layers *.Cu *.Mask)
+      (net 2 "Net-(C1-Pad2)"))
+    (pad 3 thru_hole oval (at 0 5.08) (size 1.6 1.6) (drill 0.8) (layers *.Cu *.Mask)
+      (net 103 "Net-(FUZZ_IN1-Pad2)"))
+    (pad 7 thru_hole oval (at 7.62 2.54) (size 1.6 1.6) (drill 0.8) (layers *.Cu *.Mask)
+      (net 12 +9V))
+    (pad 4 thru_hole oval (at 0 7.62) (size 1.6 1.6) (drill 0.8) (layers *.Cu *.Mask)
+      (net 5 GND))
+    (pad 8 thru_hole oval (at 7.62 0) (size 1.6 1.6) (drill 0.8) (layers *.Cu *.Mask)
+      (net 104 "Net-(U3-Pad8)"))
+    (model ${KISYS3DMOD}/Package_DIP.3dshapes/DIP-8_W7.62mm_Socket.wrl
+      (at (xyz 0 0 0))
+      (scale (xyz 1 1 1))
+      (rotate (xyz 0 0 0))
+    )
   )
   (module Capacitor_THT:CP_Radial_D10.0mm_P5.00mm (layer F.Cu)
@@
       (net 5 GND))
     (pad 2 thru_hole circle (at 5.08 0) (size 3.50012 3.50012) (drill 1.50114) (layers *.Cu *.Mask)
-      (net 2 "Net-(C1-Pad2)"))
+      (net 103 "Net-(FUZZ_IN1-Pad2)"))
   )
   (module Connector_Wire:SolderWirePad_1x02_P5.08mm_Drill1.5mm (layer F.Cu)

Commit message: Remove DAC circuit
Parts:
- removed GLIDE_POT1: Conn_01x03_Male, Connector_Wire:SolderWirePad_1x03_P4.445mm_Drill1.5mm
- removed R1: 10k, Resistor_THT:R_Axial_DIN0207_L6.3mm_D2.5mm_P10.16mm_Horizontal
- removed R2: 5K, Resistor_THT:R_Axial_DIN0207_L6.3mm_D2.5mm_P10.16mm_Horizontal
- removed R3: 150, Resistor_THT:R_Axial_DIN0207_L6.3mm_D2.5mm_P10.16mm_Horizontal
- removed U1: LM358, Package_DIP:DIP-8_W7.62mm_Socket
- removed U2: Teensy3.6, Teensy:Teensy35_36
