File: DAC/DAC.kicad_pcb (KiCad board)
At the start: 2 copper layers, 54.6 x 45.7 mm, 12 parts, among them J1 GLIDE_POT, J2 DAC_OUT, J3 9V_IN, J4 5V_IN, U1 LM358, U2 Teensy3.2

Commit message: not sure what this is tbh
Connections:
- U2 pad 32: Net-(U2-Pad32) -> GND
- U2 pad 33: Net-(U2-Pad33) -> Net-(J4-Pad2)
- U2 pad 34: Net-(J4-Pad2) -> Net-(U2-Pad34)
Routing:
- net GND: track 66.7 -> 75.7 mm
- net Net-(J4-Pad2): track 17.9 -> 9.94 mm
