File: DAC/DAC.sch (KiCad schematic (older format))
At the start: 4 parts

Commit message: Board is laid out
Parts:
- removed R?: R, symbol Device:R
- added J1: GLIDE_POT, Connector_Wire:SolderWirePad_1x03_P3.175mm_Drill1mm, symbol Connector:Conn_01x03_Male
- added J3: 9V_IN, Connector_Wire:SolderWirePad_1x02_P3.81mm_Drill1mm, symbol Connector:Conn_01x02_Male
- added J4: 5V_IN, Connector_Wire:SolderWirePad_1x02_P3.81mm_Drill1mm, symbol Connector:Conn_01x02_Male
- added R2: 9.1k, Resistor_THT:R_Axial_DIN0207_L6.3mm_D2.5mm_P10.16mm_Horizontal, symbol Device:R
- added R3: 910, Resistor_THT:R_Axial_DIN0207_L6.3mm_D2.5mm_P10.16mm_Horizontal, symbol Device:R
- added R4: 130, Resistor_THT:R_Axial_DIN0207_L6.3mm_D2.5mm_P10.16mm_Horizontal, symbol Device:R
- added R5: 20, Resistor_THT:R_Axial_DIN0207_L6.3mm_D2.5mm_P10.16mm_Horizontal, symbol Device:R
- added R6: 5.1k, Resistor_THT:R_Axial_DIN0207_L6.3mm_D2.5mm_P10.16mm_Horizontal, symbol Device:R
- added U1: LM358, Package_DIP:DIP-8_W7.62mm, symbol Amplifier_Operational:LM358
- J2: renamed from J?; footprint (none) -> Connector_Wire:SolderWirePad_1x02_P3.81mm_Drill1mm
- R1: renamed from R?; value R -> 100; footprint (none) -> Resistor_THT:R_Axial_DIN0207_L6.3mm_D2.5mm_P10.16mm_Horizontal
- U2: renamed from U?; footprint (none) -> teensy:Teensy30_31_32_LC_Rev
Connections:
- net GND: now also J2.1 (Pin_1), J1.1 (Pin_1), J4.1 (Pin_1), R3.2
- net NOTE: now reaches U2.19 (A14/DAC)
- net NOTE: now also U1.3 (+)
- net GLIDE_IN: now reaches U2.29 (22_A8_Touch_PWM)
- net GLIDE_IN: now also J1.2 (Pin_2)
- net 3.3V: now reaches U2.31 (3.3V_max100mA)
- net 3.3V: now also J1.3 (Pin_3)
- net at U2.34 (VUSB): now also J4.2 (Pin_2)
- net at J2.2 (Pin_2): now also R6.1, U1.1
- net at R1.1: now also R4.2, U1.2 (-)
- net at R1.2: now also R2.1
- new net: J3.1 (Pin_1), U1.4 (V-)
- new net: J3.2 (Pin_2), U1.8 (V+)
- new net: R4.1, R5.2
- new net: R5.1, R6.2
- new net: R2.2, R3.1
Other:
- moved on the sheet: J2, R1

Commit message: not sure what this is tbh
Connections:
- net GND: now also U2.32 (AGND)
- net at U2.33 (Vin): now also J4.2 (Pin_2)
- net at U2.34 (VUSB): no longer J4.2 (Pin_2)
Changed lines of the file:
@@
 Wire Wire Line
 	5850 3750 5850 3400
-Wire Wire Line
-	5850 3300 5850 3150
-Wire Wire Line
-	5850 3150 5100 3150
 $Comp
 L Device:R R2
@@
 Wire Wire Line
 	5400 3650 5100 3650
+$Comp
+L power:GND #PWR?
+U 1 1 5C9B8E20
+P 5700 3350
+F 0 "#PWR?" H 5700 3100 50  0001 C CNN
+F 1 "GND" H 5705 3177 50  0000 C CNN
+F 2 "" H 5700 3350 50  0001 C CNN
+F 3 "" H 5700 3350 50  0001 C CNN
+	1    5700 3350
+	1    0    0    -1
+$EndComp
+Wire Wire Line
+	5100 3350 5700 3350
+Wire Wire Line
+	5100 3250 5850 3250
+Wire Wire Line
+	5850 3250 5850 3300
 $EndSCHEMATC
